Commit message: Initial commit: ROS2 autonomous navigation robot project

File: src/maze_robot_description/urdf/robot.urdf.xacro (robot description, xacro)
@@ -178,5 +178,5 @@
         <parent link="base_link"/>
         <child link="right_wheel_link"/>
-        <origin xyz="${-base_length/3} ${-(base_width/2 + wheel_height/2)} 0" rpy="0 0 0"/>
+        <origin xyz="0 ${-(base_width/2 + wheel_height/2)} 0" rpy="0 0 0"/>
         <axis xyz="0 1 0"/>
     </joint>
@@ -184,5 +184,5 @@
         <parent link="base_link"/>
         <child link="left_wheel_link"/>
-        <origin xyz="${-base_length/3} ${(base_width/2 + wheel_height/2)} 0" rpy="0 0 0"/>
+        <origin xyz="0 ${(base_width/2 + wheel_height/2)} 0" rpy="0 0 0"/>
         <axis xyz="0 1 0"/>
     </joint>
@@ -241,5 +241,6 @@
             <pose>0 0 0 0 0 0</pose>
             <visualize>true</visualize>
-            <update_rate>10</update_rate>
+            <update_rate>20</update_rate>
+            <always_on>true</always_on>
             <ray>
                 <scan>
@@ -252,6 +253,6 @@
                 </scan>
                 <range>
-                    <min>0.1</min>
-                    <max>10.0</max>
+                    <min>0.12</min>
+                    <max>15.0</max>
                     <resolution>0.01</resolution>
                 </range>
